File: PCB_Designs/SensingCircuit/Arduino Xylophone_V02.brd (EAGLE design)
At the start: 100 x 80 mm, 92 parts, among them IC1 MCP601OT, IC10 MCP601OT, IC11 MCP601OT, IC12 MCP601OT, IC13 MCP601OT, IC2 MCP601OT, IC3 MCP601OT, IC4 MCP601OT, IC5 MCP601OT, IC6 MCP601OT, IC7 MCP601OT, IC8 MCP601OT, IC9 MCP601OT, U1 ATMEGA2560AU

Commit message: working on board layout for Xylophone sensing circuit
Parts:
- removed D25: 3.3V, SparkFun-DiscreteSemi:SOD-323
- removed D26: 250mA/100V, SparkFun-DiscreteSemi:SOD-323
- removed IC1, IC10, IC11, IC12, IC13, IC2, IC3, IC4, IC5, IC6, IC7, IC8, IC9: MCP601OT, linear:SOT23-5
- removed P-13: PIEZO, Orlando:VIA
- removed R37, R38, R39: (no value), resistor:R0402
- added #1, #10, #11, #12, #2, #3, #4, #5, #6, #7, #8, #9: MCP601OT, linear:SOT23-5
- D1: value 250mA/100V -> 3.3V
- D2: value 3.3V -> 250mA/100V
- moved P-10 183.6 mm to (2.08, 73.2), turned to 90 degrees
- moved P-11 178.3 mm to (2.77, 67.3), turned to 90 degrees
- moved U1 176.8 mm to (29.6, 52.4)
- moved R30 176.2 mm to (4.93, 72.5), flipped to the bottom, turned to 270 degrees
- moved R29 175.9 mm to (12.6, 73.0), turned to 90 degrees
- moved R28 175.6 mm to (8.53, 72.7), turned to 90 degrees
- moved R32 175.4 mm to (12.2, 68.4), turned to 90 degrees
- moved R33 174.3 mm to (4.80, 67.6), flipped to the bottom, turned to 270 degrees
- moved R31 172.0 mm to (8.48, 68.2), turned to 90 degrees
- moved D19 167.5 mm to (10.4, 72.9), turned to 90 degrees
- moved D21 163.4 mm to (10.2, 68.3), turned to 90 degrees
- moved D22 162.8 mm to (5.99, 68.8), turned to 180 degrees
- moved D20 157.8 mm to (5.89, 73.7), turned to 180 degrees
- moved P-8 131.4 mm to (3.43, 21.8), turned to 90 degrees
- moved P-9 125.1 mm to (3.68, 15.1), turned to 90 degrees
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Connections:
- removed net N$49: D25.C, IC13.3, R37.1, R38.1
- removed net N$50: D26.C, R37.2
- removed net N$51: IC13.1, IC13.4
- removed net N$52: D26.A, P-13.2, R39.1
- net 5V: now also #1.5, #10.5, #11.5, #12.5, #2.5, #3.5, #4.5, #5.5, #6.5, #7.5, #8.5, #9.5; no longer IC1.5, IC10.5, IC11.5, IC12.5, IC13.5, IC2.5, IC3.5, IC4.5, IC5.5, IC6.5, IC7.5, IC8.5, IC9.5
- net GND: now also #1.2, #10.2, #11.2, #12.2, #2.2, #3.2, #4.2, #5.2, #6.2, #7.2, #8.2, #9.2, D1.A; no longer D2.A, D25.A, IC1.2, IC10.2, IC11.2, IC12.2, IC13.2, IC2.2, IC3.2, IC4.2, IC5.2, IC6.2, IC7.2, IC8.2, IC9.2, P-13.1, R38.2, R39.2
- net N$1: now also #3.3, D1.C; no longer D2.C, IC1.3
- net N$11: now also #5.1, #5.4; no longer IC3.1, IC3.4
- net N$13: now also #6.3; no longer IC4.3
- net N$15: now also #6.1, #6.4; no longer IC4.1, IC4.4
- net N$17: now also #7.3; no longer IC5.3
- net N$19: now also #7.1, #7.4; no longer IC5.1, IC5.4
- net N$2: now also D2.C; no longer D1.C
- net N$21: now also #8.3; no longer IC6.3
- net N$23: now also #8.1, #8.4; no longer IC6.1, IC6.4
- net N$25: now also #9.3; no longer IC7.3
- net N$27: now also #9.1, #9.4; no longer IC7.1, IC7.4
- net N$29: now also #10.3; no longer IC8.3
- net N$3: now also #3.1, #3.4; no longer IC1.1, IC1.4
- net N$31: now also #10.1, #10.4; no longer IC8.1, IC8.4
- net N$33: now also #11.3; no longer IC9.3
- net N$35: now also #11.1, #11.4; no longer IC9.1, IC9.4
- net N$37: now also #1.3; no longer IC10.3
- net N$39: now also #1.1, #1.4; no longer IC10.1, IC10.4
- net N$4: now also D2.A; no longer D1.A
- net N$41: now also #2.3; no longer IC11.3
- net N$43: now also #2.1, #2.4; no longer IC11.1, IC11.4
- net N$45: now also #12.3; no longer IC12.3
- net N$47: now also #12.1, #12.4; no longer IC12.1, IC12.4
- net N$5: now also #4.3; no longer IC2.3
- net N$7: now also #4.1, #4.4; no longer IC2.1, IC2.4
- net N$9: now also #5.3; no longer IC3.3
Routing:
- net N$37: track 0.00 -> 6.67 mm
- net GND: track 0.00 -> 4.45 mm
- net N$40: track 0.00 -> 3.00 mm
- net N$38: track 0.00 -> 1.61 mm
- added copper zone on layer 1, net 5V
- added copper zone on layer 16, net GND
Other:
- board size 100 x 80 mm -> 101.6 x 76.2 mm
